File: CanBusFinalICSP.brd (EAGLE design)
At the start: 51 parts, among them IC1 PIC16F872P, U1 MCP2515

Commit message: Add files via upload
Parts:
- removed Q2: (no value), SparkFun-DiscreteSemi:TO-92
- added U2: (no value), SparkFun-PowerIC:78XXL
Connections:
- net 5V: now also U2.OUT; no longer Q2.3
- net GND: now also U2.GND; no longer Q2.2
- net N$27: now also U2.IN; no longer Q2.1
Routing:
- net 5V: track 337.2 -> 345.2 mm, vias 5 -> 6
- net N$7: track 98.0 -> 93.6 mm
- net GND: track 389.2 -> 385.0 mm
- net N$27: track 17.5 -> 19.6 mm
- net N$29: track 12.2 -> 11.2 mm
- net N$19: track 71.5 -> 70.7 mm
